Commit message: add plan node option in addition to ik node for moving of robot

File: hand_publisher/urdf/urdf/panda.gz.urdf.xacro (robot description, xacro)
@@ -1,5 +1,16 @@
 <?xml version="1.0"?>
 <robot xmlns:xacro="http://www.ros.org/wiki/xacro">
-  <xacro:macro name="panda_gz_ros2_control" params="controllers_file">
+  <xacro:macro name="panda_gz_ros2_control" params="
+    controllers_file
+    initial_panda_joint1
+    initial_panda_joint2
+    initial_panda_joint3
+    initial_panda_joint4
+    initial_panda_joint5
+    initial_panda_joint6
+    initial_panda_joint7
+    initial_panda_finger_joint1
+    initial_panda_finger_joint2
+  ">
     <ros2_control name="gz_ros2_control" type="system">
       <hardware>
@@ -8,45 +19,63 @@
       <joint name="panda_joint1">
         <command_interface name="position"/>
-        <state_interface name="position"/>
+        <state_interface name="position">
+          <param name="initial_value">${initial_panda_joint1}</param>
+        </state_interface>
         <state_interface name="velocity"/>
       </joint>
       <joint name="panda_joint2">
         <command_interface name="position"/>
-        <state_interface name="position"/>
+        <state_interface name="position">
+          <param name="initial_value">${initial_panda_joint2}</param>
+        </state_interface>
         <state_interface name="velocity"/>
       </joint>
       <joint name="panda_joint3">
         <command_interface name="position"/>
-        <state_interface name="position"/>
+        <state_interface name="position">
+          <param name="initial_value">${initial_panda_joint3}</param>
+        </state_interface>
         <state_interface name="velocity"/>
       </joint>
       <joint name="panda_joint4">
         <command_interface name="position"/>
-        <state_interface name="position"/>
+        <state_interface name="position">
+          <param name="initial_value">${initial_panda_joint4}</param>
+        </state_interface>
         <state_interface name="velocity"/>
       </joint>
       <joint name="panda_joint5">
         <command_interface name="position"/>
-        <state_interface name="position"/>
+        <state_interface name="position">
+          <param name="initial_value">${initial_panda_joint5}</param>
+        </state_interface>
         <state_interface name="velocity"/>
       </joint>
       <joint name="panda_joint6">
         <command_interface name="position"/>
-        <state_interface name="position"/>
+        <state_interface name="position">
+          <param name="initial_value">${initial_panda_joint6}</param>
+        </state_interface>
         <state_interface name="velocity"/>
       </joint>
       <joint name="panda_joint7">
         <command_interface name="position"/>
-        <state_interface name="position"/>
+        <state_interface name="position">
+          <param name="initial_value">${initial_panda_joint7}</param>
+        </state_interface>
         <state_interface name="velocity"/>
       </joint>
       <joint name="panda_finger_joint1">
         <command_interface name="position"/>
-        <state_interface name="position"/>
+        <state_interface name="position">
+          <param name="initial_value">${initial_panda_finger_joint1}</param>
+        </state_interface>
         <state_interface name="velocity"/>
       </joint>
       <joint name="panda_finger_joint2">
         <command_interface name="position"/>
-        <state_interface name="position"/>
+        <state_interface name="position">
+          <param name="initial_value">${initial_panda_finger_joint2}</param>
+        </state_interface>
         <state_interface name="velocity"/>
       </joint>

File: hand_publisher/urdf/urdf/panda.urdf.xacro (robot description, xacro)
@@ -9,4 +9,13 @@
     <xacro:arg name="use_gz" default="false"/>
     <xacro:arg name="controllers_file" default=""/>
+    <xacro:arg name="initial_panda_joint1" default="0.0"/>
+    <xacro:arg name="initial_panda_joint2" default="-0.785"/>
+    <xacro:arg name="initial_panda_joint3" default="0.0"/>
+    <xacro:arg name="initial_panda_joint4" default="-2.356"/>
+    <xacro:arg name="initial_panda_joint5" default="0.0"/>
+    <xacro:arg name="initial_panda_joint6" default="1.571"/>
+    <xacro:arg name="initial_panda_joint7" default="0.785"/>
+    <xacro:arg name="initial_panda_finger_joint1" default="0.04"/>
+    <xacro:arg name="initial_panda_finger_joint2" default="0.04"/>
     <xacro:arg name="enable_ee_camera" default="true"/>
     <xacro:arg name="enable_base_camera" default="true"/>
@@ -301,4 +310,13 @@
         <xacro:panda_gz_ros2_control
             controllers_file="$(arg controllers_file)"
+            initial_panda_joint1="$(arg initial_panda_joint1)"
+            initial_panda_joint2="$(arg initial_panda_joint2)"
+            initial_panda_joint3="$(arg initial_panda_joint3)"
+            initial_panda_joint4="$(arg initial_panda_joint4)"
+            initial_panda_joint5="$(arg initial_panda_joint5)"
+            initial_panda_joint6="$(arg initial_panda_joint6)"
+            initial_panda_joint7="$(arg initial_panda_joint7)"
+            initial_panda_finger_joint1="$(arg initial_panda_finger_joint1)"
+            initial_panda_finger_joint2="$(arg initial_panda_finger_joint2)"
         />
         <xacro:if value="$(arg enable_ee_camera)">
